Commit message: Add TurtleBot3 Lid Control and Detection Features
- Implemented LidController node for controlling the lid's position via a ROS service.
- Created LidDetector node to process camera images for potential lid detection.
- Developed a test suite (LidTester) to validate the opening and closing of the lid through service calls.
- Updated package.xml to include necessary dependencies for the new functionality.
- Added URDF and XACRO files for the lid and storage box, integrating them into the TurtleBot3 model.
- Configured Gazebo plugins for joint control and simulation of the lid.
- Created launch files to facilitate the deployment of the TurtleBot3 with the lid in a Gazebo environment.

File: turtlebot3_gazebo/urdf/turtlebot3_waffle_pi.urdf (robot description, URDF)
Before this commit: robot turtlebot3_waffle_pi, 11 links, 10 joints
Links:
- added link lid_link, mass 0.3; collision box size=0.25 0.20 0.05; visual box size=0.25 0.20 0.05
- added link storage_box_link, mass 0.5; collision box size=0.25 0.20 0.10; visual box size=0.25 0.20 0.10
Joints:
- added joint lid_joint: type revolute, parent storage_box_link, child lid_link, origin xyz=-0.125 0 0.10 rpy=0 0 0, axis 0 1 0, limit lower=0 upper=1.5708 effort=50 velocity=2.0
- added joint storage_box_joint: type fixed, parent base_link, child storage_box_link, origin xyz=-0.08 0 0.16 rpy=0 0 0

Commit message: hello

File: turtlebot3_gazebo/urdf/turtlebot3_waffle_pi.urdf (robot description, URDF)
Before this commit: robot turtlebot3_waffle_pi, 13 links, 12 joints
Links:
- link camera_link: geometry collision box size=0.015 0.030 0.027; visual box size=0.015 0.030 0.027
Joints:
- joint lid_joint: axis 0 1 0 -> 0 -1 0
- joint storage_box_joint: origin xyz=-0.08 0 0.16 rpy=0 0 0 -> xyz=-0.08 0 0.095 rpy=0 0 0
