Commit message: hello

File: rostut/urdf/robocore.urdf.xacro (robot description, xacro)
@@ -150,5 +150,5 @@
     <parent link="base_link"/>
     <child link="box"/>
-    <origin xyz="0 0 0.2" rpy="0 0 0"/>
+    <origin xyz="0 0 0.3" rpy="0 0 0"/>
 </joint>
 <link name="box">
@@ -198,3 +198,65 @@
     </collision>
 </link>
+<!-- Camera -->
+<joint name="camera_joint" type="fixed">
+    <parent link="base_link"/>
+    <child link="camera"/>
+    <origin xyz="0.5 0 0.1" rpy="0 0 0"/>
+</joint>
+<link name="camera">
+    <inertial>
+        <mass value="0.1"/>
+        <inertia ixx="0.001" ixy="0.0" ixz="0.0" iyy="0.001" iyz="0.0" izz="0.001"/>
+    </inertial>
+    <visual>
+        <origin xyz="0 0 0" rpy="0 0 0"/>
+        <geometry>
+            <box size="0.05 0.08 0.06"/>
+        </geometry>
+        <material name="dark_grey"/>
+    </visual>
+    <collision>
+        <origin xyz="0 0 0" rpy="0 0 0"/>
+        <geometry>
+            <box size="0.05 0.08 0.06"/>
+        </geometry>
+    </collision>
+</link>
+<!-- Camera RGB Optical Frame -->
+<joint name="camera_rgb_joint" type="fixed">
+    <parent link="camera"/>
+    <child link="camera_rgb_optical_frame"/>
+    <origin xyz="0.025 0 0" rpy="-1.5708 0 -1.5708"/>
+</joint>
+<link name="camera_rgb_optical_frame">
+    <inertial>
+        <mass value="0.001"/>
+        <inertia ixx="0.0001" ixy="0.0" ixz="0.0" iyy="0.0001" iyz="0.0" izz="0.0001"/>
+    </inertial>
+</link>
+<!-- Lidar -->
+<joint name="lidar_joint" type="fixed">
+    <parent link="base_link"/>
+    <child link="lidar"/>
+    <origin xyz="0 0 0.2" rpy="0 0 0"/>
+</joint>
+<link name="lidar">
+    <inertial>
+        <mass value="0.5"/>
+        <inertia ixx="0.01" ixy="0.0" ixz="0.0" iyy="0.01" iyz="0.0" izz="0.01"/>
+    </inertial>
+    <visual>
+        <origin xyz="0 0 0" rpy="0 0 0"/>
+        <geometry>
+            <cylinder radius="0.1" length="0.1"/>
+        </geometry>
+        <material name="dark_grey"/>
+    </visual>
+    <collision>
+        <origin xyz="0 0 0" rpy="0 0 0"/>
+        <geometry>
+            <cylinder radius="0.1" length="0.1"/>
+        </geometry>
+    </collision>
+</link>
 </robot>
