Commit message: hello

File: rostut/urdf/robot.urdf.xacro (robot description, xacro)
@@ -3,4 +3,7 @@
   <material name="gray">
     <color rgba="0.5 0.5 0.5 1.0"/>
+  </material>
+  <material name="red">
+    <color rgba="1 0 0 1.0"/>
   </material>
   <link name="base_link">
@@ -26,3 +29,30 @@
     </inertial>
   </link>
+  <link name="second_link">
+    <visual>
+      <geometry>
+        <box size="0.3 0.2 0.1"/>
+      </geometry>
+      <origin xyz="0 0 0.05" rpy="0 0 0"/>
+      <material name="red"/> <!-- Referencing global material -->
+    </visual>
+    <collision>
+      <geometry>
+        <box size="0.3 0.2 0.1"/>
+      </geometry>
+      <origin xyz="0 0 0.05" rpy="0 0 0"/>
+    </collision>
+    <inertial>
+      <mass value="2.0"/>
+      <origin xyz="0 0 0.05" rpy="0 0 0"/>
+      <inertia ixx="0.01" ixy="0.0" ixz="0.0"
+               iyy="0.01" iyz="0.0"
+               izz="0.01"/>
+    </inertial>
+  </link>
+  <joint name="base_to_second" type="fixed">
+    <parent link="base_link"/>
+    <child link="second_link"/>
+    <origin xyz="0 0 0.05" rpy="0 0 0"/>
+    <axis xyz="0 0 1"/>
 </robot>

Commit message: hello

File: rostut/urdf/robot.urdf.xacro (robot description, xacro)
@@ -1,58 +1,4 @@
 <?xml version="1.0"?>
 <robot xmlns:xacro="http://ros.org/wiki/xacro" name="my_robot">
-  <material name="gray">
-    <color rgba="0.5 0.5 0.5 1.0"/>
-  </material>
-  <material name="red">
-    <color rgba="1 0 0 1.0"/>
-  </material>
-  <link name="base_link">
-    <visual>
-      <geometry>
-        <box size="0.5 0.3 0.1"/>
-      </geometry>
-      <origin xyz="0 0 0.05" rpy="0 0 0"/>
-      <material name="gray"/> <!-- Referencing global material -->
-    </visual>
-    <collision>
-      <geometry>
-        <box size="0.5 0.3 0.1"/>
-      </geometry>
-      <origin xyz="0 0 0.05" rpy="0 0 0"/>
-    </collision>
-    <inertial>
-      <mass value="2.0"/>
-      <origin xyz="0 0 0.05" rpy="0 0 0"/>
-      <inertia ixx="0.01" ixy="0.0" ixz="0.0"
-               iyy="0.01" iyz="0.0"
-               izz="0.01"/>
-    </inertial>
-  </link>
-  <link name="second_link">
-    <visual>
-      <geometry>
-        <box size="0.3 0.2 0.1"/>
-      </geometry>
-      <origin xyz="0 0 0.05" rpy="0 0 0"/>
-      <material name="red"/> <!-- Referencing global material -->
-    </visual>
-    <collision>
-      <geometry>
-        <box size="0.3 0.2 0.1"/>
-      </geometry>
-      <origin xyz="0 0 0.05" rpy="0 0 0"/>
-    </collision>
-    <inertial>
-      <mass value="2.0"/>
-      <origin xyz="0 0 0.05" rpy="0 0 0"/>
-      <inertia ixx="0.01" ixy="0.0" ixz="0.0"
-               iyy="0.01" iyz="0.0"
-               izz="0.01"/>
-    </inertial>
-  </link>
-  <joint name="base_to_second" type="fixed">
-    <parent link="base_link"/>
-    <child link="second_link"/>
-    <origin xyz="0 0 0.05" rpy="0 0 0"/>
-    <axis xyz="0 0 1"/>
+<xacro:include filename="$(find rostut)/urdf/robocore.urdf.xacro"/>
 </robot>

Commit message: hello

File: rostut/urdf/robot.urdf.xacro (robot description, xacro)
@@ -1,4 +1,4 @@
 <?xml version="1.0"?>
 <robot xmlns:xacro="http://ros.org/wiki/xacro" name="my_robot">
-<xacro:include filename="$(find rostut)/urdf/robocore.urdf.xacro"/>
+<xacro:include filename="$(find rostut)/urdf/tank.urdf.xacro"/>
 </robot>

File: rostut/urdf/tank.urdf.xacro (robot description, xacro)
@@ -16,12 +16,12 @@
     <color rgba="0.1 0.25 0.5 1"/>
 </material>
-<link name="base_link"/>
+<link name="base_footprint"/>
 <!-- Base Link -->
-<joint name="chassijoint" type="fixed">
-    <parent link="base_link"/>
-    <child link="chassi"/>
+<joint name="base_joint" type="fixed">
+    <parent link="base_footprint"/>
+    <child link="base_link"/>
     <origin xyz="0.5 0 0" rpy="0 0 0"/>
 </joint>
-<link name="chassi">
+<link name="base_link">
     <visual>
         <origin xyz="0 0 0.1" rpy="0 0 0"/>
@@ -34,5 +34,5 @@
 <!-- Left Back Wheel -->
 <joint name="lbwheel_joint" type="continuous">
-    <parent link="chassi"/>
+    <parent link="base_link"/>
     <child link="lbwheel"/>
     <origin xyz="-0.4 0.3 0.1" rpy="-${pi/2} 0 0"/>
@@ -50,5 +50,5 @@
 <!-- Left Front Wheel -->
 <joint name="lfwheel_joint" type="continuous">
-    <parent link="chassi"/>
+    <parent link="base_link"/>
     <child link="lfwheel"/>
     <origin xyz="0.4 0.3 0.1" rpy="-${pi/2} 0 0"/>
@@ -66,5 +66,5 @@
 <!-- Right Front Wheel -->
 <joint name="rfwheel_joint" type="continuous">
-    <parent link="chassi"/>
+    <parent link="base_link"/>
     <child link="rfwheel"/>
     <origin xyz="0.4 -0.3 0.1" rpy="-${pi/2} 0 0"/>
@@ -82,5 +82,5 @@
 <!-- Right Back Wheel -->
 <joint name="rbwheel_joint" type="continuous">
-    <parent link="chassi"/>
+    <parent link="base_link"/>
     <child link="rbwheel"/>
     <origin xyz="-0.4 -0.3 0.1" rpy="-${pi/2} 0 0"/>
@@ -98,5 +98,5 @@
 <!-- Shooter base -->
 <joint name="shooter_joint" type="fixed">
-    <parent link="chassi"/>
+    <parent link="base_link"/>
     <child link="shooter_base"/>
     <origin xyz="0 0 0.2" rpy="0 0 0"/>
@@ -141,10 +141,10 @@
         <geometry>
           <!--  <cylinder radius="0.05" length="0.65"/> -->
-          <mesh filename="package://rostut/models/barrel.stl" scale="1 1 1"/>
+          <mesh filename="package://rostut/models/shooter/meshes/barrel.stl" scale="1 1 1"/>
         </geometry>
         <collision>
             <origin xyz="0 0 0.0" rpy="0 0 0"/>
             <geometry>
-                <mesh filename="package://rostut/models/barrel.stl" scale="1 1 1"/>
+                <mesh filename="package://rostut/models/shooter/meshes/barrel.stl" scale="1 1 1"/>
             </geometry>
         </collision>
